File: KiCadSource/file56785EF9.sch (KiCad schematic (older format))
At the start: 45 parts, among them U3 AD8337, U4 AD8337, U5 ADA4932-1, U6 ADA4932-1, U7 LTC6754

Commit message: first production run, digital GPIOs, replaced parts (see CHANGES.txt)
Parts:
- C29, C30, C31, C32: Description MLCC - SMD/SMT 0402 50V X7R 10% -> MLCC - SMD/SMT 0402 10V X7R 10%
- C33, C34: footprint ScopefunPackagesLibrary:0603 -> ScopefunPackagesLibrary:C_0603; Description MLCC - SMD/SMT 0603 50V C0G 0.25P -> MLCC - SMD/SMT 0603 100V C0G 0.25P
Changed lines of the file:
@@
 F 3 "" H 7010 2870 50  0001 C CNN
 F 4 "885012205012" H 7110 2970 60  0001 C CNN "MFG Part#"
-F 5 "MLCC - SMD/SMT 0402 50V X7R 10%" H 7050 3050 60  0001 C CNN "Description"
+F 5 "MLCC - SMD/SMT 0402 10V X7R 10%" H 7050 3050 60  0001 C CNN "Description"
 	1    7000 2800
 	1    0    0    -1
@@
 F 3 "" H 7010 970 50  0001 C CNN
 F 4 "885012205012" H 7110 1070 60  0001 C CNN "MFG Part#"
-F 5 "MLCC - SMD/SMT 0402 50V X7R 10%" H 7050 1150 60  0001 C CNN "Description"
+F 5 "MLCC - SMD/SMT 0402 10V X7R 10%" H 7050 1150 60  0001 C CNN "Description"
 	1    7000 900
 	1    0    0    -1
@@
 F 3 "" H 7010 4420 50  0001 C CNN
 F 4 "885012205012" H 7110 4520 60  0001 C CNN "MFG Part#"
-F 5 "MLCC - SMD/SMT 0402 50V X7R 10%" H 7050 4600 60  0001 C CNN "Description"
+F 5 "MLCC - SMD/SMT 0402 10V X7R 10%" H 7050 4600 60  0001 C CNN "Description"
 	1    7000 4350
 	1    0    0    -1
@@
 F 3 "" H 7060 6320 50  0001 C CNN
 F 4 "885012205012" H 7160 6420 60  0001 C CNN "MFG Part#"
-F 5 "MLCC - SMD/SMT 0402 50V X7R 10%" H 7100 6500 60  0001 C CNN "Description"
+F 5 "MLCC - SMD/SMT 0402 10V X7R 10%" H 7100 6500 60  0001 C CNN "Description"
 	1    7050 6250
 	1    0    0    -1
@@
 F 0 "C33" H 8160 1820 50  0000 L CNN
 F 1 "C_2p" H 8160 1670 50  0000 L CNN
-F 2 "ScopefunPackagesLibrary:0603" H 8150 1550 50  0001 C CNN
+F 2 "ScopefunPackagesLibrary:C_0603" H 8150 1550 50  0001 C CNN
 F 3 "" H 8160 1820 50  0001 C CNN
 F 4 "C1608C0G2A020C080AA" H 8150 1950 60  0001 C CNN "MFG Part#"
-F 5 "MLCC - SMD/SMT 0603 50V C0G 0.25P" H 8150 2050 60  0001 C CNN "Description"
+F 5 "MLCC - SMD/SMT 0603 100V C0G 0.25P" H 8150 2050 60  0001 C CNN "Description"
 	1    8150 1750
 	1    0    0    -1
@@
 F 0 "C34" H 8160 5270 50  0000 L CNN
 F 1 "C_2p" H 8160 5120 50  0000 L CNN
-F 2 "ScopefunPackagesLibrary:0603" H 8150 5000 50  0001 C CNN
+F 2 "ScopefunPackagesLibrary:C_0603" H 8150 5000 50  0001 C CNN
 F 3 "" H 8160 5270 50  0001 C CNN
 F 4 "C1608C0G2A020C080AA" H 8150 5400 60  0001 C CNN "MFG Part#"
-F 5 "MLCC - SMD/SMT 0603 50V C0G 0.25P" H 8150 5500 60  0001 C CNN "Description"
+F 5 "MLCC - SMD/SMT 0603 100V C0G 0.25P" H 8150 5500 60  0001 C CNN "Description"
 	1    8150 5200
 	1    0    0    -1
