File: KiCadSource/file56921512.sch (KiCad schematic (older format))
At the start: 46 parts, among them U10 KAD5510P-25Q48, U11 LTC6957-2, U8 KAD5510P-25Q48, U9 SG3225VAN-250Mhz

Commit message: first production run, digital GPIOs, replaced parts (see CHANGES.txt)
Parts:
- C60, C61, C62, C64, C65, C66, C67, C68: Description MLCC - SMD/SMT 0402 50V X7R 10% -> MLCC - SMD/SMT 0402 10V X7R 10%
Changed lines of the file:
@@
 F 3 "" H 6710 5220 50  0001 C CNN
 F 4 "885012205012" H 6810 5320 60  0001 C CNN "MFG Part#"
-F 5 "MLCC - SMD/SMT 0402 50V X7R 10%" H 6750 5400 60  0001 C CNN "Description"
+F 5 "MLCC - SMD/SMT 0402 10V X7R 10%" H 6750 5400 60  0001 C CNN "Description"
 	1    6700 5150
 	0    -1   -1   0
@@
 F 3 "" H 6710 5520 50  0001 C CNN
 F 4 "885012205012" H 6810 5620 60  0001 C CNN "MFG Part#"
-F 5 "MLCC - SMD/SMT 0402 50V X7R 10%" H 6750 5700 60  0001 C CNN "Description"
+F 5 "MLCC - SMD/SMT 0402 10V X7R 10%" H 6750 5700 60  0001 C CNN "Description"
 	1    6700 5450
 	0    -1   -1   0
@@
 F 3 "" H 9510 5570 50  0001 C CNN
 F 4 "885012205012" H 9610 5670 60  0001 C CNN "MFG Part#"
-F 5 "MLCC - SMD/SMT 0402 50V X7R 10%" H 9550 5750 60  0001 C CNN "Description"
+F 5 "MLCC - SMD/SMT 0402 10V X7R 10%" H 9550 5750 60  0001 C CNN "Description"
 	1    9500 5500
 	0    -1   -1   0
@@
 F 3 "" H 9510 5870 50  0001 C CNN
 F 4 "885012205012" H 9610 5970 60  0001 C CNN "MFG Part#"
-F 5 "MLCC - SMD/SMT 0402 50V X7R 10%" H 9550 6050 60  0001 C CNN "Description"
+F 5 "MLCC - SMD/SMT 0402 10V X7R 10%" H 9550 6050 60  0001 C CNN "Description"
 	1    9500 5800
 	0    -1   -1   0
@@
 F 3 "" H 9510 4870 50  0001 C CNN
 F 4 "885012205012" H 9610 4970 60  0001 C CNN "MFG Part#"
-F 5 "MLCC - SMD/SMT 0402 50V X7R 10%" H 9550 5050 60  0001 C CNN "Description"
+F 5 "MLCC - SMD/SMT 0402 10V X7R 10%" H 9550 5050 60  0001 C CNN "Description"
 	1    9500 4800
 	0    -1   -1   0
@@
 F 3 "" H 9510 5170 50  0001 C CNN
 F 4 "885012205012" H 9610 5270 60  0001 C CNN "MFG Part#"
-F 5 "MLCC - SMD/SMT 0402 50V X7R 10%" H 9550 5350 60  0001 C CNN "Description"
+F 5 "MLCC - SMD/SMT 0402 10V X7R 10%" H 9550 5350 60  0001 C CNN "Description"
 	1    9500 5100
 	0    -1   -1   0
@@
 F 3 "" H 5060 6070 50  0001 C CNN
 F 4 "885012205012" H 5160 6170 60  0001 C CNN "MFG Part#"
-F 5 "MLCC - SMD/SMT 0402 50V X7R 10%" H 5100 6250 60  0001 C CNN "Description"
+F 5 "MLCC - SMD/SMT 0402 10V X7R 10%" H 5100 6250 60  0001 C CNN "Description"
 	1    5050 6000
 	0    1    1    0
@@
 F 3 "" H 7660 4670 50  0001 C CNN
 F 4 "885012205012" H 7760 4770 60  0001 C CNN "MFG Part#"
-F 5 "MLCC - SMD/SMT 0402 50V X7R 10%" H 7700 4850 60  0001 C CNN "Description"
+F 5 "MLCC - SMD/SMT 0402 10V X7R 10%" H 7700 4850 60  0001 C CNN "Description"
 	1    7650 4600
 	0    1    1    0
