File: KiCadSource/file56948067.sch (KiCad schematic (older format))
At the start: 26 parts, among them Q3 BSS138BKS, U12 XC7A35T-FTG256

Commit message: first production run, digital GPIOs, replaced parts (see CHANGES.txt)
Parts:
- LED1, LED2, LED3: Description SMD LED “598 SERIES” 0805 PACKAGE 2V 130 mCd 140° YELLOW Cl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 -> SMD LED 598 SERIES 0805 2V 130 mCd 140 DEG YELLOW Clear
Changed lines of the file:
@@
 F 3 "https://media.digikey.com/pdf/Data%20Sheets/Dialight%20PDFs/598_Series_0805_Pkg.pdf" H 4250 6400 50  0001 C CNN
 F 4 "598-8150-107F" H 4200 7050 60  0001 C CNN "MFG Part#"
-F 5 "SMD LED “598 SERIES” 0805 PACKAGE 2V 130 mCd 140° YELLOW Clear" H 4250 7200 60  0001 C CNN "Description"
+F 5 "SMD LED 598 SERIES 0805 2V 130 mCd 140 DEG YELLOW Clear" H 4250 7200 60  0001 C CNN "Description"
 	1    4250 6750
 	1    0    0    -1
@@
 F 3 "https://media.digikey.com/pdf/Data%20Sheets/Dialight%20PDFs/598_Series_0805_Pkg.pdf" H 4250 7100 50  0001 C CNN
 F 4 "598-8150-107F" H 4200 7750 60  0001 C CNN "MFG Part#"
-F 5 "SMD LED “598 SERIES” 0805 PACKAGE 2V 130 mCd 140° YELLOW Clear" H 4250 7900 60  0001 C CNN "Description"
+F 5 "SMD LED 598 SERIES 0805 2V 130 mCd 140 DEG YELLOW Clear" H 4250 7900 60  0001 C CNN "Description"
 	1    4250 7450
 	1    0    0    -1
@@
 F 3 "https://media.digikey.com/pdf/Data%20Sheets/Dialight%20PDFs/598_Series_0805_Pkg.pdf" H 6550 6750 50  0001 C CNN
 F 4 "598-8150-107F" H 6500 7400 60  0001 C CNN "MFG Part#"
-F 5 "SMD LED “598 SERIES” 0805 PACKAGE 2V 130 mCd 140° YELLOW Clear" H 6550 7550 60  0001 C CNN "Description"
+F 5 "SMD LED 598 SERIES 0805 2V 130 mCd 140 DEG YELLOW Clear" H 6550 7550 60  0001 C CNN "Description"
 	1    6550 7100
 	1    0    0    -1
