File: KiCadSource/file584BA872.sch (KiCad schematic (older format))
At the start: 54 parts, among them U14 SN74AUP1T17DCKR, U29 CYUSB3014, U30 M24M02-DR, X1 X_Crystal_19.2Mhz

Commit message: first production run, digital GPIOs, replaced parts (see CHANGES.txt)
Parts:
- R61: Description RES SMD 1% 1/10W 0805 -> RES SMD ZERO OHM JUMPER 0805
- X1: Description Quartz crystal 19.2 Mhz -> Quartz crystal 19.2 Mhz 10ppm
