File: KiCadSource/file584EFEB1.sch (KiCad schematic (older format))
At the start: 57 parts, among them J2 SIL6, U12 XC7A35T-FTG256

Commit message: first production run, digital GPIOs, replaced parts (see CHANGES.txt)
Parts:
- C180, C205, C206, C218: Description MLCC - SMD/SMT 1210 6.3V X5R 20% -> MLCC - SMD/SMT 1210 10V X5R 20%
- C182, C183, C184, C196, C208, C209: Description MLCC - SMD/SMT 0603 10V X7R 15% -> MLCC - SMD/SMT 0805 10V X7R 10%
- C189, C190, C191, C193, C194, C195, C197, C198, C199, C201, C202, C203, C204, C207, C214, C215, C216, C217, C219, C220, C221, C222, C223: Description MLCC - SMD/SMT 0603 6.3V X7R 10% -> MLCC - SMD/SMT 0603 16V X7R 10%
