File: KiCadSource/file5855FC3A.sch (KiCad schematic (older format))
At the start: 20 parts, among them U31 DAC5662

Commit message: first production run, digital GPIOs, replaced parts (see CHANGES.txt)
Parts:
- C226: Description MLCC - SMD/SMT 0603 10V X7R 10% -> MLCC - SMD/SMT 0603 6.3V X5R 10%
- C228, C229: footprint ScopefunPackagesLibrary:0603 -> ScopefunPackagesLibrary:C_0603
Changed lines of the file:
@@
 DAC_CLK_2
 $Comp
-L GND #PWR0353
+L GND #PWR0352
 U 1 1 58595396
 P 5550 2200
-F 0 "#PWR0353" H 5550 1950 50  0001 C CNN
+F 0 "#PWR0352" H 5550 1950 50  0001 C CNN
 F 1 "GND" H 5550 2050 50  0000 C CNN
 F 2 "" H 5550 2200 50  0000 C CNN
@@
 Connection ~ 5400 1650
 $Comp
-L GND #PWR0354
+L GND #PWR0353
 U 1 1 585964D1
 P 5850 2000
-F 0 "#PWR0354" H 5850 1750 50  0001 C CNN
+F 0 "#PWR0353" H 5850 1750 50  0001 C CNN
 F 1 "GND" H 5850 1850 50  0000 C CNN
 F 2 "" H 5850 2000 50  0000 C CNN
@@
 	5300 3050 5600 3050
 $Comp
-L GND #PWR0355
+L GND #PWR0354
 U 1 1 5859A984
 P 6250 3100
-F 0 "#PWR0355" H 6250 2850 50  0001 C CNN
+F 0 "#PWR0354" H 6250 2850 50  0001 C CNN
 F 1 "GND" H 6250 2950 50  0000 C CNN
 F 2 "" H 6250 3100 50  0000 C CNN
@@
 	6500 1950 6800 1950
 $Comp
-L GND #PWR0356
+L GND #PWR0355
 U 1 1 58A69C2F
 P 6800 2000
-F 0 "#PWR0356" H 6800 1750 50  0001 C CNN
+F 0 "#PWR0355" H 6800 1750 50  0001 C CNN
 F 1 "GND" H 6800 1850 50  0000 C CNN
 F 2 "" H 6800 2000 50  0000 C CNN
@@
 	5400 1650 5400 1850
 $Comp
-L +3.3V_VA #PWR0357
+L +3.3V_VA #PWR0356
 U 1 1 58A6B1CD
 P 7450 1550
-F 0 "#PWR0357" H 7450 1400 50  0001 C CNN
+F 0 "#PWR0356" H 7450 1400 50  0001 C CNN
 F 1 "+3.3V_VA" H 7450 1690 50  0000 C CNN
 F 2 "" H 7450 1550 50  0000 C CNN
@@
 $EndComp
 $Comp
-L +3.3V #PWR0358
+L +3.3V #PWR0357
 U 1 1 58A6B2E4
 P 8700 1550
-F 0 "#PWR0358" H 8700 1400 50  0001 C CNN
+F 0 "#PWR0357" H 8700 1400 50  0001 C CNN
 F 1 "+3.3V" H 8700 1690 50  0000 C CNN
 F 2 "" H 8700 1550 50  0000 C CNN
@@
 $EndComp
 $Comp
-L +3.3V_VA #PWR0359
+L +3.3V_VA #PWR0358
 U 1 1 58A6B37F
 P 6800 1550
-F 0 "#PWR0359" H 6800 1400 50  0001 C CNN
+F 0 "#PWR0358" H 6800 1400 50  0001 C CNN
 F 1 "+3.3V_VA" H 6800 1690 50  0000 C CNN
 F 2 "" H 6800 1550 50  0000 C CNN
@@
 	6800 1550 6800 1700
 $Comp
-L +3.3V_VA #PWR0360
+L +3.3V_VA #PWR0359
 U 1 1 58A737BA
 P 5500 2800
-F 0 "#PWR0360" H 5500 2650 50  0001 C CNN
+F 0 "#PWR0359" H 5500 2650 50  0001 C CNN
 F 1 "+3.3V_VA" H 5500 2940 50  0000 C CNN
 F 2 "" H 5500 2800 50  0000 C CNN
@@
 Connection ~ 6150 1650
 $Comp
-L +3.3V_VA #PWR0361
+L +3.3V_VA #PWR0360
 U 1 1 58A74A4D
 P 5750 3900
-F 0 "#PWR0361" H 5750 3750 50  0001 C CNN
+F 0 "#PWR0360" H 5750 3750 50  0001 C CNN
 F 1 "+3.3V_VA" H 5750 4040 50  0000 C CNN
 F 2 "" H 5750 3900 50  0000 C CNN
@@
 F 3 "" H 5860 1870 50  0001 C CNN
 F 4 "C0603C105K9PACTU" H 5960 1970 60  0001 C CNN "MFG Part#"
-F 5 "MLCC - SMD/SMT 0603 10V X7R 10%" H 5900 2050 60  0001 C CNN "Description"
+F 5 "MLCC - SMD/SMT 0603 6.3V X5R 10%" H 5900 2050 60  0001 C CNN "Description"
 	1    5850 1800
 	1    0    0    -1
@@
 1.25V_REF
 $Comp
-L +Va #PWR0362
+L +Va #PWR0361
 U 1 1 58BA611F
 P 3900 5300
-F 0 "#PWR0362" H 3950 5350 50  0001 C CNN
+F 0 "#PWR0361" H 3950 5350 50  0001 C CNN
 F 1 "+Va" H 3915 5473 50  0000 C CNN
 F 2 "" H -5300 4050 50  0000 C CNN
@@
 	3900 5300 3900 5500
 $Comp
-L +Va #PWR0363
+L +Va #PWR0362
 U 1 1 58BA6132
 P 4700 5750
-F 0 "#PWR0363" H 4750 5800 50  0001 C CNN
+F 0 "#PWR0362" H 4750 5800 50  0001 C CNN
 F 1 "+Va" H 4715 5923 50  0000 C CNN
 F 2 "" H -4500 4500 50  0000 C CNN
@@
 Connection ~ 4300 5750
 $Comp
-L GND #PWR0364
+L GND #PWR0363
 U 1 1 58BA6149
 P 4300 5900
-F 0 "#PWR0364" H 4300 5650 50  0001 C CNN
+F 0 "#PWR0363" H 4300 5650 50  0001 C CNN
 F 1 "GND" H 4300 5750 50  0000 C CNN
 F 2 "" H 4300 5900 50  0000 C CNN
@@
 $EndComp
 $Comp
-L GND #PWR0365
+L GND #PWR0364
 U 1 1 58BA614F
 P 3900 5900
-F 0 "#PWR0365" H 3900 5650 50  0001 C CNN
+F 0 "#PWR0364" H 3900 5650 50  0001 C CNN
 F 1 "GND" H 3900 5750 50  0000 C CNN
 F 2 "" H 3900 5900 50  0000 C CNN
@@
 	5300 6100 5300 6000
 $Comp
-L GND #PWR0366
+L GND #PWR0365
 U 1 1 58BA6167
 P 5100 6200
-F 0 "#PWR0366" H 5100 5950 50  0001 C CNN
+F 0 "#PWR0365" H 5100 5950 50  0001 C CNN
 F 1 "GND" H 5100 6050 50  0000 C CNN
 F 2 "" H 5100 6200 50  0000 C CNN
@@
 F 0 "C228" H 6260 2670 50  0000 L CNN
 F 1 "C_0603" H 6260 2520 50  0000 L CNN
-F 2 "ScopefunPackagesLibrary:0603" H 6250 2450 50  0001 C CNN
+F 2 "ScopefunPackagesLibrary:C_0603" H 6250 2450 50  0001 C CNN
 F 3 "" H 6260 2670 50  0001 C CNN
 F 4 "Not populated" H 6250 2750 50  0001 C CNN "Description"
@@
 F 0 "C229" H 6260 3670 50  0000 L CNN
 F 1 "C_0603" H 6260 3520 50  0000 L CNN
-F 2 "ScopefunPackagesLibrary:0603" H 6250 3450 50  0001 C CNN
+F 2 "ScopefunPackagesLibrary:C_0603" H 6250 3450 50  0001 C CNN
 F 3 "" H 6260 3670 50  0001 C CNN
 F 4 "Not populated" H 6250 3750 50  0001 C CNN "Description"
