File: KiCadSource/file58568C5C.sch (KiCad schematic (older format))
At the start: 23 parts, among them U32 AZ4558C, U33 MAX5501, U34 OPA692, U35 OPA692

Commit message: first production run, digital GPIOs, replaced parts (see CHANGES.txt)
Parts:
- C237: Description MLCC - SMD/SMT 0402 50V X7R 10% -> MLCC - SMD/SMT 0402 10V X7R 10%
Changed lines of the file:
@@
 NoConn ~ 3450 2500
 $Comp
-L GND #PWR0367
+L GND #PWR0366
 U 1 1 5856C0BA
 P 3350 3400
-F 0 "#PWR0367" H 3350 3150 50  0001 C CNN
+F 0 "#PWR0366" H 3350 3150 50  0001 C CNN
 F 1 "GND" H 3350 3250 50  0000 C CNN
 F 2 "" H 3350 3400 50  0000 C CNN
@@
 $EndComp
 $Comp
-L GND #PWR0368
+L GND #PWR0367
 U 1 1 58577D66
 P 4200 5200
-F 0 "#PWR0368" H 4200 4950 50  0001 C CNN
+F 0 "#PWR0367" H 4200 4950 50  0001 C CNN
 F 1 "GND" H 4200 5050 50  0000 C CNN
 F 2 "" H 4200 5200 50  0000 C CNN
@@
 $EndComp
 $Comp
-L GND #PWR0369
+L GND #PWR0368
 U 1 1 58577D97
 P 4200 6800
-F 0 "#PWR0369" H 4200 6550 50  0001 C CNN
+F 0 "#PWR0368" H 4200 6550 50  0001 C CNN
 F 1 "GND" H 4200 6650 50  0000 C CNN
 F 2 "" H 4200 6800 50  0000 C CNN
@@
 $EndComp
 $Comp
-L GND #PWR0370
+L GND #PWR0369
 U 1 1 585A889B
 P 4850 1900
-F 0 "#PWR0370" H 4850 1650 50  0001 C CNN
+F 0 "#PWR0369" H 4850 1650 50  0001 C CNN
 F 1 "GND" H 4850 1750 50  0000 C CNN
 F 2 "" H 4850 1900 50  0000 C CNN
@@
 $EndComp
 $Comp
-L +Va #PWR0371
+L +Va #PWR0370
 U 1 1 58AA27EB
 P 9200 2000
-F 0 "#PWR0371" H 9250 2050 50  0001 C CNN
+F 0 "#PWR0370" H 9250 2050 50  0001 C CNN
 F 1 "+Va" H 9215 2173 50  0000 C CNN
 F 2 "" H 0   750 50  0000 C CNN
@@
 $EndComp
 $Comp
-L +Va #PWR0372
+L +Va #PWR0371
 U 1 1 58AA35BB
 P 3050 4150
-F 0 "#PWR0372" H 3100 4200 50  0001 C CNN
+F 0 "#PWR0371" H 3100 4200 50  0001 C CNN
 F 1 "+Va" H 3065 4323 50  0000 C CNN
 F 2 "" H -6150 2900 50  0000 C CNN
@@
 $EndComp
 $Comp
-L +Va #PWR0373
+L +Va #PWR0372
 U 1 1 58AA42D0
 P 950 1000
-F 0 "#PWR0373" H 1000 1050 50  0001 C CNN
+F 0 "#PWR0372" H 1000 1050 50  0001 C CNN
 F 1 "+Va" H 965 1173 50  0000 C CNN
 F 2 "" H -8250 -250 50  0000 C CNN
@@
 $EndComp
 $Comp
-L GND #PWR0374
+L GND #PWR0373
 U 1 1 58B1F191
 P 7250 2300
-F 0 "#PWR0374" H 7250 2050 50  0001 C CNN
+F 0 "#PWR0373" H 7250 2050 50  0001 C CNN
 F 1 "GND" H 7250 2150 50  0000 C CNN
 F 2 "" H 7250 2300 50  0000 C CNN
@@
 $EndComp
 $Comp
-L GND #PWR0375
+L GND #PWR0374
 U 1 1 58B21247
 P 7250 4300
-F 0 "#PWR0375" H 7250 4050 50  0001 C CNN
+F 0 "#PWR0374" H 7250 4050 50  0001 C CNN
 F 1 "GND" H 7250 4150 50  0000 C CNN
 F 2 "" H 7250 4300 50  0000 C CNN
@@
 CH1_OFFSET_ADJ
 $Comp
-L +3.3V_VA #PWR0376
+L +3.3V_VA #PWR0375
 U 1 1 58B27810
 P 4550 1550
-F 0 "#PWR0376" H 50  400 50  0001 C CNN
+F 0 "#PWR0375" H 50  400 50  0001 C CNN
 F 1 "+3.3V_VA" H 4565 1723 50  0000 C CNN
 F 2 "" H 50  550 50  0000 C CNN
@@
 	9000 4450 9800 4450
 $Comp
-L +Va #PWR0377
+L +Va #PWR0376
 U 1 1 58B9CD9C
 P 9200 4000
-F 0 "#PWR0377" H 9250 4050 50  0001 C CNN
+F 0 "#PWR0376" H 9250 4050 50  0001 C CNN
 F 1 "+Va" H 9215 4173 50  0000 C CNN
 F 2 "" H 0   2750 50  0000 C CNN
@@
 NoConn ~ 9000 4900
 $Comp
-L -Va #PWR0378
+L -Va #PWR0377
 U 1 1 58B9E33C
 P 9200 5000
-F 0 "#PWR0378" H 9200 4900 50  0001 C CNN
+F 0 "#PWR0377" H 9200 4900 50  0001 C CNN
 F 1 "-Va" H 9200 5140 50  0000 C CNN
 F 2 "" H 9200 5000 50  0000 C CNN
@@
 	9200 4700 9000 4700
 $Comp
-L -Va #PWR0379
+L -Va #PWR0378
 U 1 1 58B9E95B
 P 9200 3000
-F 0 "#PWR0379" H 9200 2900 50  0001 C CNN
+F 0 "#PWR0378" H 9200 2900 50  0001 C CNN
 F 1 "-Va" H 9200 3140 50  0000 C CNN
 F 2 "" H 9200 3000 50  0000 C CNN
@@
 	9200 2700 9000 2700
 $Comp
-L +Va #PWR0380
+L +Va #PWR0379
 U 1 1 58B95373
 P 1750 1450
-F 0 "#PWR0380" H 1800 1500 50  0001 C CNN
+F 0 "#PWR0379" H 1800 1500 50  0001 C CNN
 F 1 "+Va" H 1765 1623 50  0000 C CNN
 F 2 "" H -7450 200 50  0000 C CNN
@@
 Connection ~ 1350 1450
 $Comp
-L GND #PWR0381
+L GND #PWR0380
 U 1 1 58B9824C
 P 1350 1600
-F 0 "#PWR0381" H 1350 1350 50  0001 C CNN
+F 0 "#PWR0380" H 1350 1350 50  0001 C CNN
 F 1 "GND" H 1350 1450 50  0000 C CNN
 F 2 "" H 1350 1600 50  0000 C CNN
@@
 $EndComp
 $Comp
-L GND #PWR0382
+L GND #PWR0381
 U 1 1 58B98358
 P 950 1600
-F 0 "#PWR0382" H 950 1350 50  0001 C CNN
+F 0 "#PWR0381" H 950 1350 50  0001 C CNN
 F 1 "GND" H 950 1450 50  0000 C CNN
 F 2 "" H 950 1600 50  0000 C CNN
@@
 	2350 1800 2350 1700
 $Comp
-L GND #PWR0383
+L GND #PWR0382
 U 1 1 58B9A4E4
 P 2150 1900
-F 0 "#PWR0383" H 2150 1650 50  0001 C CNN
+F 0 "#PWR0382" H 2150 1650 50  0001 C CNN
 F 1 "GND" H 2150 1750 50  0000 C CNN
 F 2 "" H 2150 1900 50  0000 C CNN
@@
 F 3 "" H 5210 1820 50  0001 C CNN
 F 4 "885012205012" H 5200 1950 60  0001 C CNN "MFG Part#"
-F 5 "MLCC - SMD/SMT 0402 50V X7R 10%" H 5200 2050 60  0001 C CNN "Description"
+F 5 "MLCC - SMD/SMT 0402 10V X7R 10%" H 5200 2050 60  0001 C CNN "Description"
 	1    5200 1750
 	1    0    0    -1
 $EndComp
 $Comp
-L GND #PWR0384
+L GND #PWR0383
 U 1 1 58BB5B84
 P 5200 1900
-F 0 "#PWR0384" H 5200 1650 50  0001 C CNN
+F 0 "#PWR0383" H 5200 1650 50  0001 C CNN
 F 1 "GND" H 5200 1750 50  0000 C CNN
 F 2 "" H 5200 1900 50  0000 C CNN
@@
 	5200 1850 5200 1900
 $Comp
-L -Va #PWR0385
+L -Va #PWR0384
 U 1 1 58BBA329
 P 3050 5150
-F 0 "#PWR0385" H 3050 5050 50  0001 C CNN
+F 0 "#PWR0384" H 3050 5050 50  0001 C CNN
 F 1 "-Va" H 3050 5290 50  0000 C CNN
 F 2 "" H 3050 5150 50  0000 C CNN
@@
 $EndComp
 $Comp
-L +Va #PWR0386
+L +Va #PWR0385
 U 1 1 58BBC4D6
 P 3050 5750
-F 0 "#PWR0386" H 3100 5800 50  0001 C CNN
+F 0 "#PWR0385" H 3100 5800 50  0001 C CNN
 F 1 "+Va" H 3065 5923 50  0000 C CNN
 F 2 "" H -6150 4500 50  0000 C CNN
@@
 	3050 5750 3050 5900
 $Comp
-L -Va #PWR0387
+L -Va #PWR0386
 U 1 1 58BBC507
 P 3050 6750
-F 0 "#PWR0387" H 3050 6650 50  0001 C CNN
+F 0 "#PWR0386" H 3050 6650 50  0001 C CNN
 F 1 "-Va" H 3050 6890 50  0000 C CNN
 F 2 "" H 3050 6750 50  0000 C CNN
