File: KiCadSource/file58589F31.sch (KiCad schematic (older format))
At the start: 20 parts

Commit message: first production run, digital GPIOs, replaced parts (see CHANGES.txt)
Parts:
- C241, C242, C243: Description MLCC - SMD/SMT 0603 6.3V X5R 20% -> MLCC - SMD/SMT 0603 6.3V X5R 10%
Changed lines of the file:
@@
 F 3 "" H 3910 3620 50  0001 C CNN
 F 4 "GRM188R60J106KE47D" H 4010 3720 60  0001 C CNN "MFG Part#"
-F 5 "MLCC - SMD/SMT 0603 6.3V X5R 20%" H 3950 3800 60  0001 C CNN "Description"
+F 5 "MLCC - SMD/SMT 0603 6.3V X5R 10%" H 3950 3800 60  0001 C CNN "Description"
 	1    3900 3550
 	1    0    0    -1
@@
 F 3 "" H 3910 5370 50  0001 C CNN
 F 4 "GRM188R60J106KE47D" H 4010 5470 60  0001 C CNN "MFG Part#"
-F 5 "MLCC - SMD/SMT 0603 6.3V X5R 20%" H 3950 5550 60  0001 C CNN "Description"
+F 5 "MLCC - SMD/SMT 0603 6.3V X5R 10%" H 3950 5550 60  0001 C CNN "Description"
 	1    3900 5300
 	1    0    0    -1
@@
 $EndComp
 $Comp
-L GND #PWR0388
+L GND #PWR0387
 U 1 1 5858A61C
 P 2800 5000
-F 0 "#PWR0388" H 2800 4750 50  0001 C CNN
+F 0 "#PWR0387" H 2800 4750 50  0001 C CNN
 F 1 "GND" H 2800 4850 50  0000 C CNN
 F 2 "" H 2800 5000 50  0000 C CNN
@@
 $EndComp
 $Comp
-L GND #PWR0389
+L GND #PWR0388
 U 1 1 5858A622
 P 3450 4050
-F 0 "#PWR0389" H 3450 3800 50  0001 C CNN
+F 0 "#PWR0388" H 3450 3800 50  0001 C CNN
 F 1 "GND" H 3450 3900 50  0000 C CNN
 F 2 "" H 3450 4050 50  0000 C CNN
@@
 $EndComp
 $Comp
-L +2.88V #PWR0390
+L +2.88V #PWR0389
 U 1 1 5858A628
 P 3900 3050
-F 0 "#PWR0390" H 3900 2950 50  0001 C CNN
+F 0 "#PWR0389" H 3900 2950 50  0001 C CNN
 F 1 "+2.88V" H 3900 3190 50  0000 C CNN
 F 2 "" H 3900 3050 50  0000 C CNN
@@
 $EndComp
 $Comp
-L -2.88V #PWR0391
+L -2.88V #PWR0390
 U 1 1 5858A62E
 P 4300 5600
-F 0 "#PWR0391" H 4300 5450 50  0001 C CNN
+F 0 "#PWR0390" H 4300 5450 50  0001 C CNN
 F 1 "-2.88V" H 4300 5740 50  0000 C CNN
 F 2 "" H 4300 5600 50  0000 C CNN
@@
 $EndComp
 $Comp
-L +VCC_USB_P #PWR0392
+L +VCC_USB_P #PWR0391
 U 1 1 5858AAC9
 P 2550 1350
-F 0 "#PWR0392" H 2550 1200 50  0001 C CNN
+F 0 "#PWR0391" H 2550 1200 50  0001 C CNN
 F 1 "+VCC_USB_P" H 2550 1490 50  0000 C CNN
 F 2 "" H 2550 1350 50  0000 C CNN
@@
 $EndComp
 $Comp
-L GND #PWR0393
+L GND #PWR0392
 U 1 1 5858AB2C
 P 3450 2350
-F 0 "#PWR0393" H 3450 2100 50  0001 C CNN
+F 0 "#PWR0392" H 3450 2100 50  0001 C CNN
 F 1 "GND" H 3450 2200 50  0000 C CNN
 F 2 "" H 3450 2350 50  0000 C CNN
@@
 $EndComp
 $Comp
-L +3.3V_PD #PWR0394
+L +3.3V_PD #PWR0393
 U 1 1 5858AB3E
 P 3900 1350
-F 0 "#PWR0394" H 3900 1200 50  0001 C CNN
+F 0 "#PWR0393" H 3900 1200 50  0001 C CNN
 F 1 "+3.3V_PD" H 3900 1490 50  0000 C CNN
 F 2 "" H 3900 1350 50  0000 C CNN
@@
 	2650 3150 2550 3150
 $Comp
-L PWR_FLAG #FLG0395
+L PWR_FLAG #FLG0394
 U 1 1 5858BAB0
 P 8300 1550
-F 0 "#FLG0395" H 8300 1645 50  0001 C CNN
+F 0 "#FLG0394" H 8300 1645 50  0001 C CNN
 F 1 "PWR_FLAG" H 8300 1750 50  0000 C CNN
 F 2 "" H 8300 1550 50  0000 C CNN
@@
 $EndComp
 $Comp
-L +3.3V_PD #PWR0396
+L +3.3V_PD #PWR0395
 U 1 1 5858BAB6
 P 8300 1350
-F 0 "#PWR0396" H 8300 1200 50  0001 C CNN
+F 0 "#PWR0395" H 8300 1200 50  0001 C CNN
 F 1 "+3.3V_PD" H 8300 1490 50  0000 C CNN
 F 2 "" H 8300 1350 50  0000 C CNN
@@
 $EndComp
 $Comp
-L PWR_FLAG #FLG0397
+L PWR_FLAG #FLG0396
 U 1 1 5858BABC
 P 8800 1550
-F 0 "#FLG0397" H 8800 1645 50  0001 C CNN
+F 0 "#FLG0396" H 8800 1645 50  0001 C CNN
 F 1 "PWR_FLAG" H 8800 1750 50  0000 C CNN
 F 2 "" H 8800 1550 50  0000 C CNN
@@
 $EndComp
 $Comp
-L PWR_FLAG #FLG0398
+L PWR_FLAG #FLG0397
 U 1 1 5858BAC2
 P 9300 1550
-F 0 "#FLG0398" H 9300 1645 50  0001 C CNN
+F 0 "#FLG0397" H 9300 1645 50  0001 C CNN
 F 1 "PWR_FLAG" H 9300 1750 50  0000 C CNN
 F 2 "" H 9300 1550 50  0000 C CNN
@@
 $EndComp
 $Comp
-L -2.88V #PWR0399
+L -2.88V #PWR0398
 U 1 1 5858BAC8
 P 9300 1350
-F 0 "#PWR0399" H 9300 1200 50  0001 C CNN
+F 0 "#PWR0398" H 9300 1200 50  0001 C CNN
 F 1 "-2.88V" H 9300 1490 50  0000 C CNN
 F 2 "" H 9300 1350 50  0000 C CNN
@@
 $EndComp
 $Comp
-L +2.88V #PWR0400
+L +2.88V #PWR0399
 U 1 1 5858BACE
 P 8800 1350
-F 0 "#PWR0400" H 8800 1250 50  0001 C CNN
+F 0 "#PWR0399" H 8800 1250 50  0001 C CNN
 F 1 "+2.88V" H 8800 1490 50  0000 C CNN
 F 2 "" H 8800 1350 50  0000 C CNN
@@
 F 3 "" H 6710 1920 50  0001 C CNN
 F 4 "GRM188R60J106KE47D" H 6810 2020 60  0001 C CNN "MFG Part#"
-F 5 "MLCC - SMD/SMT 0603 6.3V X5R 20%" H 6750 2100 60  0001 C CNN "Description"
+F 5 "MLCC - SMD/SMT 0603 6.3V X5R 10%" H 6750 2100 60  0001 C CNN "Description"
 	1    6700 1850
 	1    0    0    -1
@@
 $EndComp
 $Comp
-L GND #PWR0401
+L GND #PWR0400
 U 1 1 5858E589
 P 6150 2350
-F 0 "#PWR0401" H 6150 2100 50  0001 C CNN
+F 0 "#PWR0400" H 6150 2100 50  0001 C CNN
 F 1 "GND" H 6150 2200 50  0000 C CNN
 F 2 "" H 6150 2350 50  0000 C CNN
@@
 $EndComp
 $Comp
-L +1.48V #PWR0402
+L +1.48V #PWR0401
 U 1 1 58592C5E
 P 6700 1350
-F 0 "#PWR0402" H 6700 1250 50  0001 C CNN
+F 0 "#PWR0401" H 6700 1250 50  0001 C CNN
 F 1 "+1.48V" H 6700 1490 50  0000 C CNN
 F 2 "" H 6700 1350 50  0000 C CNN
@@
 $EndComp
 $Comp
-L PWR_FLAG #FLG0403
+L PWR_FLAG #FLG0402
 U 1 1 585930EE
 P 9750 1550
-F 0 "#FLG0403" H 9750 1645 50  0001 C CNN
+F 0 "#FLG0402" H 9750 1645 50  0001 C CNN
 F 1 "PWR_FLAG" H 9750 1750 50  0000 C CNN
 F 2 "" H 9750 1550 50  0000 C CNN
@@
 	9750 1350 9750 1550
 $Comp
-L +1.48V #PWR0404
+L +1.48V #PWR0403
 U 1 1 58593126
 P 9750 1350
-F 0 "#PWR0404" H 9750 1250 50  0001 C CNN
+F 0 "#PWR0403" H 9750 1250 50  0001 C CNN
 F 1 "+1.48V" H 9750 1490 50  0000 C CNN
 F 2 "" H 9750 1350 50  0000 C CNN
@@
 $EndComp
 $Comp
-L -Va #PWR0405
+L -Va #PWR0404
 U 1 1 588596A8
 P 2550 5600
-F 0 "#PWR0405" H 2550 5500 50  0001 C CNN
+F 0 "#PWR0404" H 2550 5500 50  0001 C CNN
 F 1 "-Va" H 2550 5740 50  0000 C CNN
 F 2 "" H 2550 5600 50  0000 C CNN
@@
 	5250 1450 5250 1350
 $Comp
-L +Va #PWR0406
+L +Va #PWR0405
 U 1 1 5885966C
 P 2550 3050
-F 0 "#PWR0406" H 2550 2950 50  0001 C CNN
+F 0 "#PWR0405" H 2550 2950 50  0001 C CNN
 F 1 "+Va" H 2550 3190 50  0000 C CNN
 F 2 "" H 2550 3050 50  0000 C CNN
@@
 $EndComp
 $Comp
-L +Va #PWR0407
+L +Va #PWR0406
 U 1 1 5885B280
 P 5250 1350
-F 0 "#PWR0407" H 5250 1250 50  0001 C CNN
+F 0 "#PWR0406" H 5250 1250 50  0001 C CNN
 F 1 "+Va" H 5250 1490 50  0000 C CNN
 F 2 "" H 5250 1350 50  0000 C CNN
