File: KiCadSource/file58597EF4.sch (KiCad schematic (older format))
At the start: 27 parts, among them U36 IS43TR16256A-125KBL

Commit message: first production run, digital GPIOs, replaced parts (see CHANGES.txt)
Parts:
- C250: Description MLCC - SMD/SMT 0603 10V X7R 10% -> MLCC - SMD/SMT 0603 6.3V X5R 10%
- U36: Description 256M X 16 BIT DDR3 SRAM -> 256M X 16 BIT DDR3 SRAM 1.5V
Changed lines of the file:
@@
 $EndDescr
 $Comp
-L +1.5V #PWR0408
+L +1.5V #PWR0407
 U 1 1 5859819D
 P 9350 2000
-F 0 "#PWR0408" H 9350 1850 50  0001 C CNN
+F 0 "#PWR0407" H 9350 1850 50  0001 C CNN
 F 1 "+1.5V" H 9350 2140 50  0000 C CNN
 F 2 "" H 9350 2000 50  0000 C CNN
@@
 $EndComp
 $Comp
-L GND #PWR0409
+L GND #PWR0408
 U 1 1 5859ADCA
 P 7800 4600
-F 0 "#PWR0409" H 7800 4350 50  0001 C CNN
+F 0 "#PWR0408" H 7800 4350 50  0001 C CNN
 F 1 "GND" H 7800 4450 50  0000 C CNN
 F 2 "" H 7800 4600 50  0000 C CNN
@@
 $EndComp
 $Comp
-L GND #PWR0410
+L GND #PWR0409
 U 1 1 5859CF1F
 P 10750 4400
-F 0 "#PWR0410" H 10750 4150 50  0001 C CNN
+F 0 "#PWR0409" H 10750 4150 50  0001 C CNN
 F 1 "GND" H 10750 4250 50  0000 C CNN
 F 2 "" H 10750 4400 50  0000 C CNN
@@
 $EndComp
 $Comp
-L GND #PWR0411
+L GND #PWR0410
 U 1 1 5859F47E
 P 4350 1750
-F 0 "#PWR0411" H 4350 1500 50  0001 C CNN
+F 0 "#PWR0410" H 4350 1500 50  0001 C CNN
 F 1 "GND" H 4350 1600 50  0000 C CNN
 F 2 "" H 4350 1750 50  0000 C CNN
@@
 DDR3_DQ15
 $Comp
-L GND #PWR0412
+L GND #PWR0411
 U 1 1 585A8A09
 P 6100 5150
-F 0 "#PWR0412" H 6100 4900 50  0001 C CNN
+F 0 "#PWR0411" H 6100 4900 50  0001 C CNN
 F 1 "GND" H 6100 5000 50  0000 C CNN
 F 2 "" H 6100 5150 50  0000 C CNN
@@
 $EndComp
 $Comp
-L GND #PWR0413
+L GND #PWR0412
 U 1 1 585AB03D
 P 6400 4050
-F 0 "#PWR0413" H 6400 3800 50  0001 C CNN
+F 0 "#PWR0412" H 6400 3800 50  0001 C CNN
 F 1 "GND" H 6400 3900 50  0000 C CNN
 F 2 "" H 6400 4050 50  0000 C CNN
@@
 DDR3_RESET#
 $Comp
-L GND #PWR0414
+L GND #PWR0413
 U 1 1 585B2A30
 P 4650 5300
-F 0 "#PWR0414" H 4650 5050 50  0001 C CNN
+F 0 "#PWR0413" H 4650 5050 50  0001 C CNN
 F 1 "GND" H 4650 5150 50  0000 C CNN
 F 2 "" H 4650 5300 50  0000 C CNN
@@
 $EndComp
 $Comp
-L +1.5V #PWR0415
+L +1.5V #PWR0414
 U 1 1 586157B0
 P 7800 3950
-F 0 "#PWR0415" H 7800 3800 50  0001 C CNN
+F 0 "#PWR0414" H 7800 3800 50  0001 C CNN
 F 1 "+1.5V" H 7800 4090 50  0000 C CNN
 F 2 "" H 7800 3950 50  0000 C CNN
@@
 $EndComp
 $Comp
-L +1.5V #PWR0416
+L +1.5V #PWR0415
 U 1 1 58615C4D
 P 8650 3950
-F 0 "#PWR0416" H 8650 3800 50  0001 C CNN
+F 0 "#PWR0415" H 8650 3800 50  0001 C CNN
 F 1 "+1.5V" H 8650 4090 50  0000 C CNN
 F 2 "" H 8650 3950 50  0000 C CNN
@@
 F 3 "" H 8310 4470 50  0001 C CNN
 F 4 "C0603C105K9PACTU" H 8410 4570 60  0001 C CNN "MFG Part#"
-F 5 "MLCC - SMD/SMT 0603 10V X7R 10%" H 8350 4650 60  0001 C CNN "Description"
+F 5 "MLCC - SMD/SMT 0603 6.3V X5R 10%" H 8350 4650 60  0001 C CNN "Description"
 	1    8300 4400
 	1    0    0    -1
@@
 $EndComp
 $Comp
-L +1.5V #PWR0417
+L +1.5V #PWR0416
 U 1 1 586D745A
 P 7650 2100
-F 0 "#PWR0417" H 7650 1950 50  0001 C CNN
+F 0 "#PWR0416" H 7650 1950 50  0001 C CNN
 F 1 "+1.5V" H 7650 2240 50  0000 C CNN
 F 2 "" H 7650 2100 50  0000 C CNN
@@
 $EndComp
 $Comp
-L GND #PWR0418
+L GND #PWR0417
 U 1 1 586D8B5B
 P 8900 2500
-F 0 "#PWR0418" H 8900 2250 50  0001 C CNN
+F 0 "#PWR0417" H 8900 2250 50  0001 C CNN
 F 1 "GND" H 8900 2350 50  0000 C CNN
 F 2 "" H 8900 2500 50  0000 C CNN
@@
 $EndComp
 $Comp
-L +1.5V #PWR0419
+L +1.5V #PWR0418
 U 1 1 586DB678
 P 7650 2800
-F 0 "#PWR0419" H 7650 2650 50  0001 C CNN
+F 0 "#PWR0418" H 7650 2650 50  0001 C CNN
 F 1 "+1.5V" H 7650 2940 50  0000 C CNN
 F 2 "" H 7650 2800 50  0000 C CNN
@@
 $EndComp
 $Comp
-L GND #PWR0420
+L GND #PWR0419
 U 1 1 586DB6B1
 P 8900 3200
-F 0 "#PWR0420" H 8900 2950 50  0001 C CNN
+F 0 "#PWR0419" H 8900 2950 50  0001 C CNN
 F 1 "GND" H 8900 3050 50  0000 C CNN
 F 2 "" H 8900 3200 50  0000 C CNN
@@
 F 3 "http://www.issi.com/WW/pdf/43-46TR16256A-85120AL.pdf" H 5450 1600 60  0001 C CNN
 F 4 "IS43TR16256A-125KBL" H 5450 1450 50  0001 C CNN "MFG Part#"
-F 5 "256M X 16 BIT DDR3 SRAM" H 5400 5200 50  0001 C CNN "Description"
+F 5 "256M X 16 BIT DDR3 SRAM 1.5V" H 5400 5200 50  0001 C CNN "Description"
 	1    5450 3450
 	1    0    0    -1
@@
 F 2 "ScopefunPackagesLibrary:TW-BGA-96" H 10000 1350 60  0001 C CNN
 F 3 "http://www.issi.com/WW/pdf/43-46TR16640B-81280BL.pdf" H 10000 1650 60  0001 C CNN
-F 4 "256M X 16 BIT DDR3 SRAM" H 9950 5250 50  0001 C CNN "Description"
+F 4 "256M X 16 BIT DDR3 SRAM 1.5V" H 9950 5250 50  0001 C CNN "Description"
 F 5 "IS43TR16640B-125JBL" H 10000 1500 50  0001 C CNN "MFG Part#"
 	2    10000 3500
